File: timeoffset.kicad_pcb (KiCad board)
At the start: 2 copper layers, 15.2 x 23.7 mm, 8 parts

Commit message: Little fixes
Other:
- board text added: "5VOUT | 5VIN | GND"
- board text added: "VCC|MOSI|GND"
- board text removed: "5VOUT | GND | 5VIN"
- board text removed: "5V|MOSI|GND"

Commit message: update
Routing:
- net Net-(C1-Pad2): vias 2 -> 0
